File: pcb/flight-computer.kicad_pcb (KiCad board)
At the start: 2 copper layers, 176 parts, among them J1 XT60PW-M, J10 Conn_01x03_Pin, J11 Conn_01x03_Pin, J12 Conn_01x03_Pin, J13 Conn_01x03_Pin, J14 Conn_01x03_Pin, J15 Conn_02x10_Counter_Clockwise, J16 3220-10-0100-00, J17 Conn_ARM_SWD_TagConnect_TC2030, J18 MSD-4-A, J19 Conn_01x04_Pin, J2 Screw_Terminal_01x02, J3 UJ20-C-H-G-SMT-P16-TR, J4 Screw_Terminal_01x02, J5 Screw_Terminal_01x02, J6 Screw_Terminal_01x02, J7 Conn_01x04_Pin_P2.54mm, J8 Conn_01x04_Qwiic, J9 Conn_01x03_Pin, Q1 NTR4003N, Q2 NTR4003N, Q3 NTR4003N, Q4 DMG2305UX, SW1 PTS815, SW2 PTS815, SW3 PTS815, SW4 PTS815, U1 STM32H523VETx, U10 BUK9K25-40RAX, U11 MC091GX, U12 Wio-SX1262, U13 W25Q128JVS, U14 MAX-M10S, U2 AP62300TWU, U3 LM66200, U4 ZXCT180B3W5, U5 TLV75733PDBV, U6 USBLC6-2SC6, U7 LPS22HH, U8 LIS2MDL, U9 LSM6DSV80X, Y1 ECS-160-12-33B2Q-JES-TR3, Y2 SC32S-7PF20PPM

Commit message: Move things around on PCB
Parts:
- moved J16 186.2 mm to (269.0, 36.0)
- moved R47 183.0 mm to (262.8, 42.4)
- moved R48 183.0 mm to (262.8, 44.9)
- moved R49 183.0 mm to (262.8, 47.5)
- moved R50 183.0 mm to (262.8, 50.0)
- moved R51 183.0 mm to (262.8, 52.5)
- moved J2 176.9 mm to (-101.0, 27.0)
- moved R55 176.1 mm to (239.5, 35.2), turned to 90 degrees
- moved R54 172.2 mm to (236.5, 35.2), turned to 90 degrees
- moved R53 172.0 mm to (238.0, 35.2), turned to 90 degrees
- moved R52 168.1 mm to (235.0, 35.2), turned to 90 degrees
- moved C23 165.9 mm to (-52.3, 16.0), turned to 180 degrees
- moved J17 161.0 mm to (238.3, 41.4)
- moved J1 154.4 mm to (-89.0, 40.0)
- moved R12 152.7 mm to (-56.5, 19.0), turned to -90 degrees
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